File: NQSAP PCB schematics/loaderV1/loader.sch (KiCad schematic (older format))
At the start: 23 parts, among them J1 Bus, J2 Bus, J5 Conn_02x08, SW1 RESET, U1 74LS173, U2 74LS173, U3 74HCT574, U4 74HCT574, U5 74HCT04, U6 74HCT08

Commit message: Add Microcode and IR/RC modules.  Add clock circuit to Loader module.
Parts:
- removed C6, C7, C8: 0.1uF, Capacitor_SMD:C_0805_2012Metric_Pad1.18x1.45mm_HandSolder, symbol Device:C
- removed U5: 74HCT04, Package_DIP:DIP-14_W7.62mm, symbol 74xx:74HCT04
- removed U6: 74HCT08, Package_DIP:DIP-14_W7.62mm, symbol 74xx:74LS08
- added U5: 74HCT00, Package_DIP:DIP-14_W7.62mm, symbol 74xx:74HCT00
- R1: value R-BLUE -> 100
- SW1: footprint Button_Switch_THT:SW_PUSH_6mm -> Button_Switch_THT:SW_PUSH_6mm_H7.3mm
Connections:
- net labels added: +5V, LDR-ACT, LDR-CLK, NC-1, NC-2, RST, ~LDR-ACT
- net labels removed: LD-ACT, LD-CLK, VCC, ~CLK, ~LD-ACT
- wire segments 271 -> 270
- no-connect marks 57 -> 54
Other:
- note added: "to control ROM2\nmisc signals"
- note added: "to control ROM3 read\nregister decoders"
- note added: "to control ROM3 write\nregister decoders"
- note removed: "Control ROM0 signals"
- note removed: "Control ROM1 signals"
- note removed: "Control ROM2\nread register selects"
- note removed: "Control ROM2\nwrite register selects"
- moved on the sheet: C1, C2, C3, C4, C5, D2, R1
