File: NQSAP PCB schematics/microcode/microcode.sch (KiCad schematic (older format))
At the start: 58 parts, among them J1 Bus, J2 Bus, J5 Conn_02x08, J6 Conn_02x08, U1 28C256, U2 28C256, U3 28C256

Commit message: Add Microcode and IR/RC modules.  Add clock circuit to Loader module.
Parts:
- added J3: IC-LT, Connector_PinHeader_2.54mm:PinHeader_1x04_P2.54mm_Vertical, symbol Connector_Generic:Conn_01x04
- J5: value Conn_02x08 -> IC-RT
- J6: value Conn_02x08 -> IC-RB
Connections:
- net labels added: CLK, ~CLK, ~RST
- wire segments 330 -> 338
- no-connect marks 27 -> 26
Other:
- moved on the sheet: C1, C2, C3
Changed lines of the file:
@@
 U 1 1 6167BE3C
 P 8200 4450
-F 0 "J5" H 8118 5067 50  0000 C CNN
-F 1 "Conn_02x08" H 8118 4976 50  0000 C CNN
+F 0 "J5" H 8100 4950 50  0000 C CNN
+F 1 "IC-RT" H 8100 4850 50  0000 C CNN
 F 2 "Connector_PinHeader_2.54mm:PinHeader_1x08_P2.54mm_Vertical" H 8200 4450 50  0001 C CNN
 F 3 "~" H 8200 4450 50  0001 C CNN
@@
 U 1 1 61847F95
 P 8200 5650
-F 0 "J6" H 8118 6267 50  0000 C CNN
-F 1 "Conn_02x08" H 8118 6176 50  0000 C CNN
+F 0 "J6" H 8100 6150 50  0000 C CNN
+F 1 "IC-RB" H 8100 6050 50  0000 C CNN
 F 2 "Connector_PinHeader_2.54mm:PinHeader_1x08_P2.54mm_Vertical" H 8200 5650 50  0001 C CNN
 F 3 "~" H 8200 5650 50  0001 C CNN
@@
 L Device:C C1
 U 1 1 640ECCCC
-P 6950 4650
-F 0 "C1" V 6800 4850 50  0000 C CNN
-F 1 "0.1uF" V 6900 4850 50  0000 C CNN
-F 2 "Capacitor_SMD:C_0805_2012Metric_Pad1.18x1.45mm_HandSolder" H 6988 4500 50  0001 C CNN
-F 3 "~" H 6950 4650 50  0001 C CNN
-	1    6950 4650
+P 1450 3750
+F 0 "C1" V 1300 3950 50  0000 C CNN
+F 1 "0.1uF" V 1400 3950 50  0000 C CNN
+F 2 "Capacitor_SMD:C_0805_2012Metric_Pad1.18x1.45mm_HandSolder" H 1488 3600 50  0001 C CNN
+F 3 "~" H 1450 3750 50  0001 C CNN
+	1    1450 3750
 	0    1    1    0
 $EndComp
@@
 L power:GND #PWR06
 U 1 1 640EE08A
-P 7300 5500
-F 0 "#PWR06" H 7300 5250 50  0001 C CNN
-F 1 "GND" H 7305 5327 50  0000 C CNN
-F 2 "" H 7300 5500 50  0001 C CNN
-F 3 "" H 7300 5500 50  0001 C CNN
-	1    7300 5500
+P 1800 4600
+F 0 "#PWR06" H 1800 4350 50  0001 C CNN
+F 1 "GND" H 1805 4427 50  0000 C CNN
+F 2 "" H 1800 4600 50  0001 C CNN
+F 3 "" H 1800 4600 50  0001 C CNN
+	1    1800 4600
 	1    0    0    -1
 $EndComp
@@
 L power:+5V #PWR05
 U 1 1 640EE95F
-P 6600 4450
-F 0 "#PWR05" H 6600 4300 50  0001 C CNN
-F 1 "+5V" H 6615 4623 50  0000 C CNN
-F 2 "" H 6600 4450 50  0001 C CNN
-F 3 "" H 6600 4450 50  0001 C CNN
-	1    6600 4450
+P 1100 3550
+F 0 "#PWR05" H 1100 3400 50  0001 C CNN
+F 1 "+5V" H 1115 3723 50  0000 C CNN
+F 2 "" H 1100 3550 50  0001 C CNN
+F 3 "" H 1100 3550 50  0001 C CNN
+	1    1100 3550
 	1    0    0    -1
 $EndComp
@@
 L power:PWR_FLAG #FLG02
 U 1 1 640EF226
-P 7300 4450
-F 0 "#FLG02" H 7300 4525 50  0001 C CNN
-F 1 "PWR_FLAG" H 7300 4623 50  0000 C CNN
-F 2 "" H 7300 4450 50  0001 C CNN
-F 3 "~" H 7300 4450 50  0001 C CNN
-	1    7300 4450
+P 1800 3550
+F 0 "#FLG02" H 1800 3625 50  0001 C CNN
+F 1 "PWR_FLAG" H 1800 3723 50  0000 C CNN
+F 2 "" H 1800 3550 50  0001 C CNN
+F 3 "~" H 1800 3550 50  0001 C CNN
+	1    1800 3550
 	1    0    0    -1
 $EndComp
@@
 L power:PWR_FLAG #FLG01
 U 1 1 640EFA22
-P 6600 5500
-F 0 "#FLG01" H 6600 5575 50  0001 C CNN
-F 1 "PWR_FLAG" H 6600 5673 50  0000 C CNN
-F 2 "" H 6600 5500 50  0001 C CNN
-F 3 "~" H 6600 5500 50  0001 C CNN
-	1    6600 5500
+P 1100 4600
+F 0 "#FLG01" H 1100 4675 50  0001 C CNN
+F 1 "PWR_FLAG" H 1100 4773 50  0000 C CNN
+F 2 "" H 1100 4600 50  0001 C CNN
+F 3 "~" H 1100 4600 50  0001 C CNN
+	1    1100 4600
 	-1   0    0    1
 $EndComp
 Wire Wire Line
-	6600 4450 6600 4650
-Wire Wire Line
-	7300 4450 7300 4650
-Wire Wire Line
-	7100 4650 7300 4650
-Connection ~ 7300 4650
-Wire Wire Line
-	7300 4650 7300 4900
-Wire Wire Line
-	6800 4650 6600 4650
-Connection ~ 6600 4650
-Wire Wire Line
-	6600 4650 6600 4900
+	1100 3550 1100 3750
+Wire Wire Line
+	1800 3550 1800 3750
+Wire Wire Line
+	1600 3750 1800 3750
+Connection ~ 1800 3750
+Wire Wire Line
+	1800 3750 1800 4000
+Wire Wire Line
+	1300 3750 1100 3750
+Connection ~ 1100 3750
+Wire Wire Line
+	1100 3750 1100 4000
 $Comp
 L Device:C C2
 U 1 1 64103212
-P 6950 4900
-F 0 "C2" V 6800 5100 50  0000 C CNN
-F 1 "0.1uF" V 6900 5100 50  0000 C CNN
-F 2 "Capacitor_SMD:C_0805_2012Metric_Pad1.18x1.45mm_HandSolder" H 6988 4750 50  0001 C CNN
-F 3 "~" H 6950 4900 50  0001 C CNN
-	1    6950 4900
+P 1450 4000
+F 0 "C2" V 1300 4200 50  0000 C CNN
+F 1 "0.1uF" V 1400 4200 50  0000 C CNN
+F 2 "Capacitor_SMD:C_0805_2012Metric_Pad1.18x1.45mm_HandSolder" H 1488 3850 50  0001 C CNN
+F 3 "~" H 1450 4000 50  0001 C CNN
+	1    1450 4000
 	0    1    1    0
 $EndComp
 Wire Wire Line
-	6800 4900 6600 4900
-Connection ~ 6600 4900
-Wire Wire Line
-	6600 4900 6600 5150
-Wire Wire Line
-	7100 4900 7300 4900
-Connection ~ 7300 4900
-Wire Wire Line
-	7300 4900 7300 5150
+	1300 4000 1100 4000
+Connection ~ 1100 4000
+Wire Wire Line
+	1100 4000 1100 4250
+Wire Wire Line
+	1600 4000 1800 4000
+Connection ~ 1800 4000
+Wire Wire Line
+	1800 4000 1800 4250
 $Comp
 L Device:C C3
 U 1 1 6410A335
-P 6950 5150
-F 0 "C3" V 6800 5350 50  0000 C CNN
-F 1 "0.1uF" V 6900 5350 50  0000 C CNN
-F 2 "Capacitor_SMD:C_0805_2012Metric_Pad1.18x1.45mm_HandSolder" H 6988 5000 50  0001 C CNN
-F 3 "~" H 6950 5150 50  0001 C CNN
-	1    6950 5150
+P 1450 4250
+F 0 "C3" V 1300 4450 50  0000 C CNN
+F 1 "0.1uF" V 1400 4450 50  0000 C CNN
+F 2 "Capacitor_SMD:C_0805_2012Metric_Pad1.18x1.45mm_HandSolder" H 1488 4100 50  0001 C CNN
+F 3 "~" H 1450 4250 50  0001 C CNN
+	1    1450 4250
 	0    1    1    0
 $EndComp
 Wire Wire Line
-	7100 5150 7300 5150
-Connection ~ 7300 5150
-Wire Wire Line
-	6800 5150 6600 5150
-Connection ~ 6600 5150
+	1600 4250 1800 4250
+Connection ~ 1800 4250
+Wire Wire Line
+	1300 4250 1100 4250
+Connection ~ 1100 4250
 $Comp
 L Memory_EEPROM:28C256 U1
@@
 Connection ~ 2050 2050
 Wire Wire Line
-	6600 5150 6600 5500
-Wire Wire Line
-	7300 5150 7300 5500
+	1100 4250 1100 4600
+Wire Wire Line
+	1800 4250 1800 4600
 Text GLabel 1000 2150 0    50   Input ~ 0
 MA6
@@
 NoConn ~ 10750 5750
 NoConn ~ 10750 5850
-NoConn ~ 9950 5850
 NoConn ~ 9950 5650
-NoConn ~ 9950 5550
 NoConn ~ 10750 3050
 NoConn ~ 10750 2950
@@
 Text GLabel 2700 1550 1    50   Output ~ 0
 WR0
+$Comp
+L Connector_Generic:Conn_01x04 J3
+U 1 1 61CEDB71
+P 7150 4250
+F 0 "J3" H 7100 4550 50  0000 C CNN
+F 1 "IC-LT" H 7100 4450 50  0000 C CNN
+F 2 "Connector_PinHeader_2.54mm:PinHeader_1x04_P2.54mm_Vertical" H 7150 4250 50  0001 C CNN
+F 3 "~" H 7150 4250 50  0001 C CNN
+	1    7150 4250
+	-1   0    0    -1
+$EndComp
+Text GLabel 8500 4450 2    50   Input ~ 0
+LD-ACT
+Text GLabel 8500 4150 2    50   Input ~ 0
+~RST
+Text GLabel 8500 4250 2    50   Input ~ 0
+~CLK
+Text GLabel 8500 4350 2    50   Input ~ 0
+CLK
+Wire Wire Line
+	8500 4150 8400 4150
+Wire Wire Line
+	8400 4250 8500 4250
+Wire Wire Line
+	8500 4350 8400 4350
+Wire Wire Line
+	8400 4450 8500 4450
+Text GLabel 7450 4450 2    50   Input ~ 0
+LD-ACT
+Text GLabel 7450 4150 2    50   Input ~ 0
+~RST
+Text GLabel 7450 4250 2    50   Input ~ 0
+~CLK
+Text GLabel 7450 4350 2    50   Input ~ 0
+CLK
+Wire Wire Line
+	7450 4150 7350 4150
+Wire Wire Line
+	7350 4250 7450 4250
+Wire Wire Line
+	7450 4350 7350 4350
+Wire Wire Line
+	7350 4450 7450 4450
+NoConn ~ 9950 5750
+Text GLabel 9950 5550 2    50   Input ~ 0
+CLK
+Text GLabel 9950 5850 2    50   Input ~ 0
+~RST
 Wire Bus Line
 	1350 1000 1350 2800
 Wire Bus Line
 	1350 2800 8250 2800
-Text GLabel 9950 5750 2    50   Input ~ 0
-LD-ACT
 $EndSCHEMATC

Commit message: Add RAM, update and add gerbers for new boards
Parts:
- D14: value XX0 -> SE
- D19: value SI -> M1
- D20: value SE -> M0
Connections:
- net labels added: M0, M1
- net labels removed: SI, XX0
- no-connect marks 26 -> 28
Other:
- moved on the sheet: J1, J2, J5, J6, U1, U2, U3
