File: NQSAP PCB schematics/backplane/backplane.kicad_pcb (KiCad board)
At the start: 2 copper layers, 360 x 128 mm, 44 parts, among them J1 Bus, J10 Bus, J11 Bus, J12 Bus, J13 Bus, J14 Bus, J15 Bus, J16 Bus, J17 Bus, J18 Bus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

Commit message: Add RAM, update and add gerbers for new boards
Connections:
- net LDR-ACT renamed ~JMP
- net LDR-CLK renamed nc3
- net NC-1 renamed nc2
- net NC-2 renamed nc1
- net RST renamed ~RST
- net SI renamed M1
- J1 pad 25: XX0 -> SE
- J1 pad 31: SE -> M0
- J10 pad 25: XX0 -> SE
- J10 pad 31: SE -> M0
- J11 pad 25: XX0 -> SE
- J11 pad 31: SE -> M0
- J12 pad 25: XX0 -> SE
- J12 pad 31: SE -> M0
- J13 pad 25: XX0 -> SE
- J13 pad 31: SE -> M0
- J14 pad 25: XX0 -> SE
- J14 pad 31: SE -> M0
- J15 pad 25: XX0 -> SE
- J15 pad 31: SE -> M0
- J16 pad 25: XX0 -> SE
- J16 pad 31: SE -> M0
- J17 pad 25: XX0 -> SE
- J17 pad 31: SE -> M0
- J18 pad 25: XX0 -> SE
- J18 pad 31: SE -> M0
- J2 pad 25: XX0 -> SE
- J2 pad 31: SE -> M0
- J3 pad 25: XX0 -> SE
- J3 pad 31: SE -> M0
- J4 pad 25: XX0 -> SE
- J4 pad 31: SE -> M0
- J5 pad 25: XX0 -> SE
- J5 pad 31: SE -> M0
- J6 pad 25: XX0 -> SE
- J6 pad 31: SE -> M0
- J7 pad 25: XX0 -> SE
- J7 pad 31: SE -> M0
- J8 pad 25: XX0 -> SE
- J8 pad 31: SE -> M0
- J9 pad 25: XX0 -> SE
- J9 pad 31: SE -> M0
Routing:
- net M0: track 0.00 -> 664.0 mm
- net XX0: track 601.1 -> 0.00 mm
- net SE: track 664.0 -> 601.1 mm

Commit message: build 5 board updates
Parts:
- added J27: POWER IN, TerminalBlock_RND:TerminalBlock_RND_205-00012_1x02_P5.00mm_Horizontal, F.Cu at (43.1, 89.1)
- added J28: POWER IN, TerminalBlock_RND:TerminalBlock_RND_205-00012_1x02_P5.00mm_Horizontal, F.Cu at (43.0, 135.6)
- added J29: POWER IN, TerminalBlock_RND:TerminalBlock_RND_205-00012_1x02_P5.00mm_Horizontal, F.Cu at (391.9, 84.1)
- added J30: POWER IN, TerminalBlock_RND:TerminalBlock_RND_205-00012_1x02_P5.00mm_Horizontal, F.Cu at (391.9, 130.7)
Other:
- board text added: "2022 rev 1.1"
- board text removed: "2021 rev 1.0"
