File: NQSAP PCB schematics/d-register/d-register.kicad_pcb (KiCad board)
At the start: 2 copper layers, 102 x 96 mm, 52 parts, among them J1 Bus, J2 Bus, J5 Conn_01x04, J6 Conn_01x08, U1 74HCT377, U2 74HCT245, U3 74LS283, U4 74LS283, U5 74HCT138, U6 74HCT138

Commit message: build 5 board updates
Connections:
- net /XY0 renamed XY0
- net /XY1 renamed XY1
- net /XY2 renamed XY2
- net /XY3 renamed XY3
- net /XY4 renamed XY4
- net /XY5 renamed XY5
- net /XY6 renamed XY6
- net /XY7 renamed XY7
