File: NQSAP PCB schematics/loader/loader.sch (KiCad schematic (older format))
At the start: 23 parts, among them J1 Bus, J2 Bus, J5 Conn_02x08, SW1 RESET, U1 74LS173, U2 74LS173, U3 74HCT574, U4 74HCT574, U5 74HCT04, U6 74HCT08

Commit message: Add RAM, update and add gerbers for new boards
Parts:
- removed C8: 0.1uF, Capacitor_SMD:C_0805_2012Metric_Pad1.18x1.45mm_HandSolder, symbol Device:C
- removed U1, U2: 74LS173, Package_DIP:DIP-16_W7.62mm, symbol 74xx:74LS173
- removed U3, U4: 74HCT574, Package_DIP:DIP-20_W7.62mm, symbol 74xx:74HCT574
- added J3: POWER IN, TerminalBlock_RND:TerminalBlock_RND_205-00012_1x02_P5.00mm_Horizontal, symbol Connector:Screw_Terminal_01x02
- added U1, U2, U3: 74HCT595, Package_SO:SOIC-16_3.9x9.9mm_P1.27mm, symbol 74xx:74HCT595
- D1: value diode -> 1N5818; footprint Diode_THT:D_DO-35_SOD27_P7.62mm_Horizontal -> Diode_THT:D_DO-41_SOD81_P10.16mm_Horizontal; symbol Device:D -> Device:D_Schottky_Small
- J5: value Conn_02x08 -> IB-TR; footprint Connector_PinHeader_2.54mm:PinHeader_1x08_P2.54mm_Vertical -> Connector_PinHeader_2.54mm:PinHeader_1x04_P2.54mm_Vertical; symbol Connector_Generic:Conn_01x08 -> Connector_Generic:Conn_01x04
Connections:
- net CLR is gone; now on net LD2: A1.19 (A0)
- net C0: now also U2.15 (QA)
- net C1: now also U2.1 (QB)
- net CC: now also U3.6 (QG)
- net CLK: no longer J2.36 (Pin_36)
- net CS: now also U3.7 (QH)
- net FB: now also U2.3 (QD)
- net FC: now also U2.4 (QE)
- net FN: now also U2.7 (QH)
- net FV: now also U2.6 (QG)
- net FZ: now also U2.5 (QF)
- net GND: now also J3.1 (Pin_1), U1.8 (GND), U2.8 (GND), U3.8 (GND)
- net JE: now also U3.2 (QC)
- net LD-CLK: now also A1.24 (A5); no longer A1.14 (D11)
- net LD0: now also U2.11 (SRCLK), U3.11 (SRCLK)
- net LD2: now also U1.11 (SRCLK); no longer A1.20 (A1)
- net LF: now also U3.3 (QD)
- net N: now also U3.1 (QB)
- net PI: now also U3.15 (QA)
- net RR0: now also U1.15 (QA)
- net RR1: now also U1.1 (QB)
- net RR2: now also U1.2 (QC)
- net RR3: now also U1.3 (QD)
- net SE: now also U3.4 (QE)
- net SI: now also U3.5 (QF)
- net VCC: now also J3.2 (Pin_2), U1.10 (~SRCLR), U1.16 (VCC), U2.10 (~SRCLR), U2.16 (VCC), U3.10 (~SRCLR), U3.16 (VCC)
- net WR0: now also U1.4 (QE)
- net WR1: now also U1.5 (QF)
- net WR2: now also U1.6 (QG)
- net WR3: now also U1.7 (QH)
- net XX0: now also U2.2 (QC)
- net ~LD-ACT: now also U1.13 (~OE), U2.13 (~OE), U3.13 (~OE)
- net ~LD-R: now also A1.23 (A4); no longer A1.15 (D12)
- net LD1 renamed RCLK
- net RCLK: now also U1.12 (RCLK), U2.12 (RCLK), U3.12 (RCLK)
- new net: U2.14 (SER), U3.9 (QH')
- new net SER: A1.20 (A1), U1.14 (SER), U3.14 (SER)
- no-connect marks 57 -> 56
Other:
- note added: "Control ROM2\nregister selects"
- note removed: "AUX"
- note removed: "Control ROM2\nread register selects"
- note removed: "Control ROM2\nwrite register selects"
- note removed: "READ"
- note removed: "WRITE"
- moved on the sheet: D1
