File: NQSAP PCB schematics/alu/alu.kicad_pcb (KiCad board)
At the start: 2 copper layers, 102 x 96 mm, 38 parts, among them J1 Bus, J2 Bus, J3 IC-TL, J4 IC-BL, J5 IC-TR, J6 IC-BR, U1 74HCT02, U2 74HCT151, U3 74HCT151, U4 74LS181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

Commit message: build 5 board updates
Parts:
- added D9: READ, LED_SMD:LED_0805_2012Metric_Pad1.15x1.40mm_HandSolder, F.Cu at (131.1, 49.0)
- added R9: R_GRN, Resistor_SMD:R_0805_2012Metric_Pad1.20x1.40mm_HandSolder, F.Cu at (135.8, 49.0)
Routing:
- net ~RL: track 86.1 -> 114.9 mm
- net Net-(D9-Pad2): track 0.00 -> 2.74 mm
- net +5V: track 30.9 -> 32.8 mm, vias 0 -> 1
Other:
- board text added: "2022 v1.1"
- board text removed: "2021 v1.0"
Changed lines of the file:
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@@
     (thickness 1.6)
     (drawings 133)
-    (tracks 690)
+    (tracks 699)
     (zones 0)
-    (modules 38)
-    (nets 152)
+    (modules 40)
+    (nets 153)
   )
   (page USLetter)
@@
   )
   (layers
-    (0 F.Cu signal hide)
-    (31 B.Cu signal)
+    (0 F.Cu signal)
+    (31 B.Cu signal hide)
     (32 B.Adhes user)
     (33 F.Adhes user)
@@
   (net 150 "Net-(J3-Pad1)")
   (net 151 "Net-(J5-Pad4)")
+  (net 152 "Net-(D9-Pad2)")
   (net_class Default "This is the default net class."
     (clearance 0.2)
@@
     (add_net "Net-(D7-Pad2)")
     (add_net "Net-(D8-Pad2)")
+    (add_net "Net-(D9-Pad2)")
     (add_net "Net-(J1-Pad12)")
     (add_net "Net-(J1-Pad13)")
@@
     (add_net ~WI)
   )
+  (module Resistor_SMD:R_0805_2012Metric_Pad1.20x1.40mm_HandSolder (layer F.Cu)
+    (at 135.845 48.955 180)
+    (descr "Resistor SMD 0805 (2012 Metric), square (rectangular) end terminal, IPC_7351 nominal with elongated pad for handsoldering. (Body size source: IPC-SM-782 page 72, https://www.pcb-3d.com/wordpress/wp-content/uploads/ipc-sm-782a_amendment_1_and_2.pdf), generated with kicad-footprint-generator")
+    (tags "resistor handsolder")
+    (attr smd)
+    (fp_text reference R9 (at -3.055 -1.245) (layer F.SilkS)
+      (effects (font (size 1 1) (thickness 0.15)))
+    )
+    (fp_text value R_GRN (at 0.045 -1.745) (layer F.Fab)
+      (effects (font (size 1 1) (thickness 0.15)))
+    )
+    (fp_line (start 1.85 0.95) (end -1.85 0.95) (layer F.CrtYd) (width 0.05))
+    (fp_line (start 1.85 -0.95) (end 1.85 0.95) (layer F.CrtYd) (width 0.05))
+    (fp_line (start -1.85 -0.95) (end 1.85 -0.95) (layer F.CrtYd) (width 0.05))
+    (fp_line (start -1.85 0.95) (end -1.85 -0.95) (layer F.CrtYd) (width 0.05))
+    (fp_line (start -0.227064 0.735) (end 0.227064 0.735) (layer F.SilkS) (width 0.12))
+    (fp_line (start -0.227064 -0.735) (end 0.227064 -0.735) (layer F.SilkS) (width 0.12))
+    (fp_line (start 1 0.625) (end -1 0.625) (layer F.Fab) (width 0.1))
+    (fp_line (start 1 -0.625) (end 1 0.625) (layer F.Fab) (width 0.1))
+    (fp_line (start -1 -0.625) (end 1 -0.625) (layer F.Fab) (width 0.1))
+    (fp_line (start -1 0.625) (end -1 -0.625) (layer F.Fab) (width 0.1))
+    (fp_text user %R (at 0 0) (layer F.Fab)
+      (effects (font (size 0.5 0.5) (thickness 0.08)))
+    )
+    (pad 2 smd roundrect (at 1 0 180) (size 1.2 1.4) (layers F.Cu F.Paste F.Mask) (roundrect_rratio 0.2083325)
+      (net 152 "Net-(D9-Pad2)"))
+    (pad 1 smd roundrect (at -1 0 180) (size 1.2 1.4) (layers F.Cu F.Paste F.Mask) (roundrect_rratio 0.2083325)
+      (net 1 +5V))
+    (model ${KISYS3DMOD}/Resistor_SMD.3dshapes/R_0805_2012Metric.wrl
+      (at (xyz 0 0 0))
+      (scale (xyz 1 1 1))
+      (rotate (xyz 0 0 0))
+    )
+  )
+  (module LED_SMD:LED_0805_2012Metric_Pad1.15x1.40mm_HandSolder (layer F.Cu)
+    (at 131.1 49)
+    (descr "LED SMD 0805 (2012 Metric), square (rectangular) end terminal, IPC_7351 nominal, (Body size source: https://docs.google.com/spreadsheets/d/1BsfQQcO9C6DZCsRaXUlFlo91Tg2WpOkGARC1WS5S8t0/edit?usp=sharing), generated with kicad-footprint-generator")
+    (tags "LED handsolder")
+    (attr smd)
+    (fp_text reference D9 (at -3.1 0) (layer F.SilkS)
+      (effects (font (size 1 1) (thickness 0.15)))
+    )
+    (fp_text value READ (at 0 2.2) (layer F.SilkS)
+      (effects (font (size 1.5 1.5) (thickness 0.17)))
+    )
+    (fp_line (start 1.85 0.95) (end -1.85 0.95) (layer F.CrtYd) (width 0.05))
+    (fp_line (start 1.85 -0.95) (end 1.85 0.95) (layer F.CrtYd) (width 0.05))
+    (fp_line (start -1.85 -0.95) (end 1.85 -0.95) (layer F.CrtYd) (width 0.05))
+    (fp_line (start -1.85 0.95) (end -1.85 -0.95) (layer F.CrtYd) (width 0.05))
+    (fp_line (start -1.86 0.96) (end 1 0.96) (layer F.SilkS) (width 0.12))
+    (fp_line (start -1.86 -0.96) (end -1.86 0.96) (layer F.SilkS) (width 0.12))
+    (fp_line (start 1 -0.96) (end -1.86 -0.96) (layer F.SilkS) (width 0.12))
+    (fp_line (start 1 0.6) (end 1 -0.6) (layer F.Fab) (width 0.1))
+    (fp_line (start -1 0.6) (end 1 0.6) (layer F.Fab) (width 0.1))
+    (fp_line (start -1 -0.3) (end -1 0.6) (layer F.Fab) (width 0.1))
+    (fp_line (start -0.7 -0.6) (end -1 -0.3) (layer F.Fab) (width 0.1))
+    (fp_line (start 1 -0.6) (end -0.7 -0.6) (layer F.Fab) (width 0.1))
+    (fp_text user %R (at 0 0) (layer F.Fab)
+      (effects (font (size 0.5 0.5) (thickness 0.08)))
+    )
+    (pad 2 smd roundrect (at 1.025 0) (size 1.15 1.4) (layers F.Cu F.Paste F.Mask) (roundrect_rratio 0.2173904347826087)
+      (net 152 "Net-(D9-Pad2)"))
+    (pad 1 smd roundrect (at -1.025 0) (size 1.15 1.4) (layers F.Cu F.Paste F.Mask) (roundrect_rratio 0.2173904347826087)
+      (net 74 ~RL))
+    (model ${KISYS3DMOD}/LED_SMD.3dshapes/LED_0805_2012Metric.wrl
+      (at (xyz 0 0 0))
+      (scale (xyz 1 1 1))
+      (rotate (xyz 0 0 0))
+    )
+  )
   (module Connector_PinHeader_2.54mm:PinHeader_2x08_P2.54mm_Vertical (layer B.Cu)
     (at 91.5 57.6 180)
@@
     )
   )
-  (gr_text "2021 v1.0" (at 185.6 94.9 90) (layer F.SilkS)
+  (gr_text "2022 v1.1" (at 185.6 94.9 90) (layer F.SilkS)
     (effects (font (size 1 1) (thickness 0.15)) (justify left))
   )
@@
   (segment (start 171.3375 79.2825) (end 171.32 79.3) (width 0.25) (layer F.Cu) (net 1))
   (segment (start 171.3375 75.2) (end 171.3375 79.2825) (width 0.25) (layer F.Cu) (net 1))
+  (via (at 138.7 49) (size 0.8) (drill 0.4) (layers F.Cu B.Cu) (net 1))
+  (segment (start 138.655 48.955) (end 138.7 49) (width 0.25) (layer F.Cu) (net 1))
+  (segment (start 136.845 48.955) (end 138.655 48.955) (width 0.25) (layer F.Cu) (net 1))
   (via (at 133.3 128.8) (size 0.8) (drill 0.4) (layers F.Cu B.Cu) (net 2))
   (segment (start 175.3 136) (end 174.124999 137.175001) (width 0.25) (layer F.Cu) (net 2))
@@
   (segment (start 107.4 66.675) (end 97.751998 66.675) (width 0.25) (layer F.Cu) (net 74))
   (segment (start 97.751998 66.675) (end 92.9 71.526998) (width 0.25) (layer F.Cu) (net 74))
+  (segment (start 130.075 49.025) (end 130.075 49) (width 0.25) (layer F.Cu) (net 74))
+  (segment (start 126.194999 52.905001) (end 130.075 49.025) (width 0.25) (layer F.Cu) (net 74))
+  (segment (start 104.465001 52.905001) (end 126.194999 52.905001) (width 0.25) (layer F.Cu) (net 74))
+  (segment (start 103.34 51.78) (end 104.465001 52.905001) (width 0.25) (layer F.Cu) (net 74))
   (via (at 184.1 104.8) (size 0.8) (drill 0.4) (layers F.Cu B.Cu) (net 114))
   (segment (start 184.1 123.18) (end 184.1 104.8) (width 0.25) (layer F.Cu) (net 114))
@@
   (segment (start 182.559002 138.1) (end 184.200001 136.459001) (width 0.25) (layer F.Cu) (net 137))
   (segment (start 184.200001 127.099999) (end 184.7 126.6) (width 0.25) (layer F.Cu) (net 137))
+  (segment (start 134.8 49) (end 134.845 48.955) (width 0.25) (layer F.Cu) (net 152))
+  (segment (start 132.125 49) (end 134.8 49) (width 0.25) (layer F.Cu) (net 152))
   (zone (net 14) (net_name GND) (layer F.Cu) (hatch edge 0.508)
     (connect_pads (clearance 0.508))
